File: SELE_ACS/SELE_ACS.kicad_pcb (KiCad board)
At the start: 2 copper layers, 20 parts, among them J1 AVR-ISP-6, J2 Input Cables, J3 FT232 Adapter, SW1 Button Reset, SW2 SW_DIP_x04, U1 atmega328p, U2 MAX485E, U3 LM7805_TO220, Y1 Crystal 8MHz

Commit message: Add files via upload
Parts:
- added REF**: MountingHole_2.2mm_M2_Pad, MountingHole:MountingHole_2.2mm_M2_Pad, F.Cu at (80.6, 107.8)
- added REF**: MountingHole_2.2mm_M2_Pad, MountingHole:MountingHole_2.2mm_M2_Pad, F.Cu at (80.6, 66.6)
- added REF**: MountingHole_2.2mm_M2_Pad, MountingHole:MountingHole_2.2mm_M2_Pad, F.Cu at (144.2, 66.6)
- moved C5 9.72 mm to (141.6, 86.2)
- moved J1 3.50 mm to (136.2, 95.9)
Routing:
- net GND: track 185.1 -> 0.00 mm
- net RX: track 40.0 -> 48.8 mm
- net SCK: track 16.9 -> 9.91 mm
- net MISO: track 6.05 -> 9.55 mm
- net RESET: track 84.4 -> 87.3 mm
- net MOSI: track 9.58 -> 12.1 mm
- net AVCC: track 85.7 -> 84.5 mm
- net TX: track 24.7 -> 25.2 mm
Other:
- board outline added: 70 x 47.5 mm
- board text added: "12V"
- board text added: "5V"
- board text added: "A"
- board text added: "B"
- board text added: "FT232"
- board text added: "GND"
- board text added: "MISO"
- board text added: "RS485"
- board text added: "RST"
- board text added: "RX"
- board text added: "SCK"
- board text added: "SELE FEUP AVR RS485 V0.1"
- board text added: "TX"
- board text added: "VCC"

Commit message: Add files via upload
gerber up
Routing:
- added copper zone on F.Cu, net GND
Changed lines of the file:
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@@
     (47 F.CrtYd user)
     (48 B.Fab user)
-    (49 F.Fab user hide)
+    (49 F.Fab user)
   )
   (setup
@@
     (visible_elements FFFFFF7F)
     (pcbplotparams
-      (layerselection 0x010fc_ffffffff)
+      (layerselection 0x010f0_ffffffff)
       (usegerberextensions false)
       (usegerberattributes false)
@@
       (outputformat 1)
       (mirror false)
-      (drillshape 1)
+      (drillshape 0)
       (scaleselection 1)
-      (outputdirectory ""))
+      (outputdirectory "GERBER/"))
   )
   (net 0 "")
@@
     (effects (font (size 1 1) (thickness 0.2)))
   )
-  (dimension 44.8 (width 0.15) (layer F.Fab)
-    (gr_text "44.800 mm" (at 152.7 88.2 270) (layer F.Fab)
-      (effects (font (size 1 1) (thickness 0.15)))
-    )
-    (feature1 (pts (xy 144.4 110.6) (xy 151.986421 110.6)))
-    (feature2 (pts (xy 144.4 65.8) (xy 151.986421 65.8)))
-    (crossbar (pts (xy 151.4 65.8) (xy 151.4 110.6)))
-    (arrow1a (pts (xy 151.4 110.6) (xy 150.813579 109.473496)))
-    (arrow1b (pts (xy 151.4 110.6) (xy 151.986421 109.473496)))
-    (arrow2a (pts (xy 151.4 65.8) (xy 150.813579 66.926504)))
-    (arrow2b (pts (xy 151.4 65.8) (xy 151.986421 66.926504)))
-  )
-  (dimension 67 (width 0.15) (layer F.Fab)
-    (gr_text "67.000 mm" (at 110.9 58.3) (layer F.Fab)
-      (effects (font (size 1 1) (thickness 0.15)))
-    )
-    (feature1 (pts (xy 144.4 65.8) (xy 144.4 59.013579)))
-    (feature2 (pts (xy 77.4 65.8) (xy 77.4 59.013579)))
-    (crossbar (pts (xy 77.4 59.6) (xy 144.4 59.6)))
-    (arrow1a (pts (xy 144.4 59.6) (xy 143.273496 60.186421)))
-    (arrow1b (pts (xy 144.4 59.6) (xy 143.273496 59.013579)))
-    (arrow2a (pts (xy 77.4 59.6) (xy 78.526504 60.186421)))
-    (arrow2b (pts (xy 77.4 59.6) (xy 78.526504 59.013579)))
+  (dimension 47.500105 (width 0.15) (layer F.Fab)
+    (gr_text "47.500 mm" (at 152.349982 87.266842 89.87937748) (layer F.Fab)
+      (effects (font (size 1 1) (thickness 0.15)))
+    )
+    (feature1 (pts (xy 144.3 111) (xy 151.586405 111.01534)))
+    (feature2 (pts (xy 144.4 63.5) (xy 151.686405 63.51534)))
+    (crossbar (pts (xy 151.099985 63.514105) (xy 150.999985 111.014105)))
+    (arrow1a (pts (xy 150.999985 111.014105) (xy 150.415937 109.886369)))
+    (arrow1b (pts (xy 150.999985 111.014105) (xy 151.588776 109.888838)))
+    (arrow2a (pts (xy 151.099985 63.514105) (xy 150.511194 64.639372)))
+    (arrow2b (pts (xy 151.099985 63.514105) (xy 151.684033 64.641841)))
+  )
+  (dimension 70.000071 (width 0.15) (layer F.Fab)
+    (gr_text "70.000 mm" (at 112.410714 58.350013 359.9181489) (layer F.Fab)
+      (effects (font (size 1 1) (thickness 0.15)))
+    )
+    (feature1 (pts (xy 147.4 65.9) (xy 147.409695 59.113592)))
+    (feature2 (pts (xy 77.4 65.8) (xy 77.409695 59.013592)))
+    (crossbar (pts (xy 77.408857 59.600012) (xy 147.408857 59.700012)))
+    (arrow1a (pts (xy 147.408857 59.700012) (xy 146.281517 60.284823)))
+    (arrow1b (pts (xy 147.408857 59.700012) (xy 146.283192 59.111983)))
+    (arrow2a (pts (xy 77.408857 59.600012) (xy 78.534522 60.188041)))
+    (arrow2b (pts (xy 77.408857 59.600012) (xy 78.536197 59.015201)))
   )
   (gr_text "SELE\nFEUP\nAVR RS485 \nV0.1" (at 80.2 97.8) (layer F.SilkS)
@@
   (segment (start 114.9 80.22) (end 119.9 80.22) (width 0.3) (layer F.Cu) (net 30))
   (segment (start 114.9 82.76) (end 114.9 80.22) (width 0.3) (layer F.Cu) (net 30))
+  (zone (net 1) (net_name GND) (layer F.Cu) (hatch edge 0.508)
+    (connect_pads (clearance 0.254))
+    (min_thickness 0.254)
+    (fill yes (arc_segments 32) (thermal_gap 0.508) (thermal_bridge_width 0.508))
+    (polygon
+      (pts
+        (xy 76.7 62.6) (xy 149.1 62.6) (xy 149.1 112) (xy 76.7 112) (xy 76.7 62.4)
+        (xy 76.7 62.5)
+      )
+    )
+  )
 )

Commit message: Add files via upload
v0.1.2
Parts:
- C1, C2: footprint Capacitor_THT:CP_Radial_D4.0mm_P1.50mm -> Capacitor_THT:C_Rect_L7.0mm_W2.0mm_P5.00mm
- moved C1 1.80 mm to (108.3, 93.0)
- moved C2 1.80 mm to (108.3, 97.9)
Routing:
- net XTAL1: track 13.4 -> 11.6 mm
- net XTAL2: track 14.4 -> 12.6 mm
- net B: track 15.6 -> 17.3 mm
- net A: track 16.3 -> 15.6 mm
Other:
- board text added: "SELE FEUP AVR RS485 V0.1.2"
- board text removed: "SELE FEUP AVR RS485 V0.1"
