File: SELE_ACS/SELE_ACS.sch (KiCad schematic (older format))
At the start: 20 parts, among them J1 AVR-ISP-6, J2 Input Cables, J3 FT232 Adapter, SW1 Button Reset, SW2 SW_DIP_x04, U1 atmega328p, U2 MAX485E, U3 LM7805_TO220, Y1 Crystal 8MHz

Commit message: Add files via upload
v0.1.2
Parts:
- C1, C2: footprint Capacitor_THT:CP_Radial_D4.0mm_P1.50mm -> Capacitor_THT:C_Rect_L7.0mm_W2.0mm_P5.00mm
Changed lines of the file:
@@
 F 0 "C1" V 4202 2300 50  0000 C CNN
 F 1 "22pF" V 4111 2300 50  0000 C CNN
-F 2 "Capacitor_THT:CP_Radial_D4.0mm_P1.50mm" H 3950 2300 50  0001 C CNN
+F 2 "Capacitor_THT:C_Rect_L7.0mm_W2.0mm_P5.00mm" H 3950 2300 50  0001 C CNN
 F 3 "~" H 3950 2300 50  0001 C CNN
 	1    3950 2300
@@
 F 0 "C2" V 3700 2600 50  0000 C CNN
 F 1 "22pF" V 3800 2600 50  0000 C CNN
-F 2 "Capacitor_THT:CP_Radial_D4.0mm_P1.50mm" H 3950 2600 50  0001 C CNN
+F 2 "Capacitor_THT:C_Rect_L7.0mm_W2.0mm_P5.00mm" H 3950 2600 50  0001 C CNN
 F 3 "~" H 3950 2600 50  0001 C CNN
 	1    3950 2600
